File: _saved_WeatherStation.sch (KiCad schematic (older format))
At the start: 14 parts, among them P1 CONN_BATT, P2 CONN_LOAD, P3 CONN_VREG, P4 CONN_FEATHER12, P5 CONN_FEATHER16, P6 CONN_RB, P7 CONN_WS, P8 CONN_RB, P9 CONN_WS, Q1 Q_NMOS_GDS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

Commit message: Fixed Gerbers
Updated the footprint pins on the Fuel Gauge
Parts:
- P8, P9: footprint Socket_Strips:Socket_Strip_Straight_1x04 -> Connectors_JST:JST_PH_B4B-PH-K_04x2.00mm_Straight
Changed lines of the file:
@@
 	7250 2050 7550 2050
 $Comp
-L +5V #PWR16
+L +5V #PWR01
 U 1 1 58879E9B
 P 7100 2150
-F 0 "#PWR16" H 7100 2000 50  0001 C CNN
+F 0 "#PWR01" H 7100 2000 50  0001 C CNN
 F 1 "+5V" H 7100 2290 50  0000 C CNN
 F 2 "" H 7100 2150 50  0000 C CNN
@@
 	7100 2150 7550 2150
 $Comp
-L +5V #PWR3
+L +5V #PWR02
 U 1 1 58879F1E
 P 2150 4350
-F 0 "#PWR3" H 2150 4200 50  0001 C CNN
+F 0 "#PWR02" H 2150 4200 50  0001 C CNN
 F 1 "+5V" H 2150 4490 50  0000 C CNN
 F 2 "" H 2150 4350 50  0000 C CNN
@@
 	2150 4350 1850 4350
 $Comp
-L GND #PWR4
+L GND #PWR03
 U 1 1 58879F81
 P 2500 4250
-F 0 "#PWR4" H 2500 4000 50  0001 C CNN
+F 0 "#PWR03" H 2500 4000 50  0001 C CNN
 F 1 "GND" H 2500 4100 50  0000 C CNN
 F 2 "" H 2500 4250 50  0000 C CNN
@@
 B+
 $Comp
-L GND #PWR2
+L GND #PWR04
 U 1 1 5887A372
 P 2000 2150
-F 0 "#PWR2" H 2000 1900 50  0001 C CNN
+F 0 "#PWR04" H 2000 1900 50  0001 C CNN
 F 1 "GND" H 2000 2000 50  0000 C CNN
 F 2 "" H 2000 2150 50  0000 C CNN
@@
 	2000 2150 1750 2150
 $Comp
-L GND #PWR14
+L GND #PWR05
 U 1 1 5887A442
 P 6100 3250
-F 0 "#PWR14" H 6100 3000 50  0001 C CNN
+F 0 "#PWR05" H 6100 3000 50  0001 C CNN
 F 1 "GND" H 6100 3100 50  0000 C CNN
 F 2 "" H 6100 3250 50  0000 C CNN
@@
 	6100 3250 6100 3150
 $Comp
-L GND #PWR15
+L GND #PWR06
 U 1 1 5887A48E
 P 6100 4350
-F 0 "#PWR15" H 6100 4100 50  0001 C CNN
+F 0 "#PWR06" H 6100 4100 50  0001 C CNN
 F 1 "GND" H 6100 4200 50  0000 C CNN
 F 2 "" H 6100 4350 50  0000 C CNN
@@
 	7350 4500 7650 4500
 $Comp
-L +5V #PWR17
+L +5V #PWR07
 U 1 1 5887A63E
 P 7200 4600
-F 0 "#PWR17" H 7200 4450 50  0001 C CNN
+F 0 "#PWR07" H 7200 4450 50  0001 C CNN
 F 1 "+5V" H 7200 4740 50  0000 C CNN
 F 2 "" H 7200 4600 50  0000 C CNN
@@
 	5250 4000 5800 4000
 $Comp
-L GND #PWR12
+L GND #PWR08
 U 1 1 5887A8FF
 P 5200 3500
-F 0 "#PWR12" H 5200 3250 50  0001 C CNN
+F 0 "#PWR08" H 5200 3250 50  0001 C CNN
 F 1 "GND" H 5200 3350 50  0000 C CNN
 F 2 "" H 5200 3500 50  0000 C CNN
@@
 	5200 3500 5200 3400
 $Comp
-L GND #PWR13
+L GND #PWR09
 U 1 1 5887A951
 P 5250 4650
-F 0 "#PWR13" H 5250 4400 50  0001 C CNN
+F 0 "#PWR09" H 5250 4400 50  0001 C CNN
 F 1 "GND" H 5250 4500 50  0000 C CNN
 F 2 "" H 5250 4650 50  0000 C CNN
@@
 	5250 4650 5250 4500
 $Comp
-L GND #PWR10
+L GND #PWR010
 U 1 1 5887ABF6
 P 4700 3950
-F 0 "#PWR10" H 4700 3700 50  0001 C CNN
+F 0 "#PWR010" H 4700 3700 50  0001 C CNN
 F 1 "GND" H 4700 3800 50  0000 C CNN
 F 2 "" H 4700 3950 50  0000 C CNN
@@
 	3350 3350 3650 3350
 $Comp
-L +5V #PWR9
+L +5V #PWR011
 U 1 1 5887AD80
 P 3400 3650
-F 0 "#PWR9" H 3400 3500 50  0001 C CNN
+F 0 "#PWR011" H 3400 3500 50  0001 C CNN
 F 1 "+5V" H 3400 3790 50  0000 C CNN
 F 2 "" H 3400 3650 50  0000 C CNN
@@
 	7650 3800 7650 4700
 $Comp
-L GND #PWR6
+L GND #PWR012
 U 1 1 5887B050
 P 2750 1200
-F 0 "#PWR6" H 2750 950 50  0001 C CNN
+F 0 "#PWR012" H 2750 950 50  0001 C CNN
 F 1 "GND" H 2750 1050 50  0000 C CNN
 F 2 "" H 2750 1200 50  0000 C CNN
@@
 NoConn ~ 4500 3350
 $Comp
-L +3V3 #PWR7
+L +3V3 #PWR013
 U 1 1 5887B4D4
 P 2850 1050
-F 0 "#PWR7" H 2850 900 50  0001 C CNN
+F 0 "#PWR013" H 2850 900 50  0001 C CNN
 F 1 "+3V3" H 2850 1190 50  0000 C CNN
 F 2 "" H 2850 1050 50  0000 C CNN
@@
 	2850 1050 3050 1050
 $Comp
-L +3V3 #PWR11
+L +3V3 #PWR014
 U 1 1 5887B682
 P 4750 4150
-F 0 "#PWR11" H 4750 4000 50  0001 C CNN
+F 0 "#PWR014" H 4750 4000 50  0001 C CNN
 F 1 "+3V3" H 4750 4290 50  0000 C CNN
 F 2 "" H 4750 4150 50  0000 C CNN
@@
 NoConn ~ 4500 3450
 $Comp
-L PWR_FLAG #FLG1
+L PWR_FLAG #FLG015
 U 1 1 5887BA33
 P 1950 6000
-F 0 "#FLG1" H 1950 6095 50  0001 C CNN
+F 0 "#FLG015" H 1950 6095 50  0001 C CNN
 F 1 "PWR_FLAG" H 1950 6180 50  0000 C CNN
 F 2 "" H 1950 6000 50  0000 C CNN
@@
 $EndComp
 $Comp
-L +5V #PWR1
+L +5V #PWR016
 U 1 1 5887BA75
 P 1950 6300
-F 0 "#PWR1" H 1950 6150 50  0001 C CNN
+F 0 "#PWR016" H 1950 6150 50  0001 C CNN
 F 1 "+5V" H 1950 6440 50  0000 C CNN
 F 2 "" H 1950 6300 50  0000 C CNN
@@
 	1950 6300 1950 6000
 $Comp
-L PWR_FLAG #FLG2
+L PWR_FLAG #FLG017
 U 1 1 5887BB48
 P 2550 6000
-F 0 "#FLG2" H 2550 6095 50  0001 C CNN
+F 0 "#FLG017" H 2550 6095 50  0001 C CNN
 F 1 "PWR_FLAG" H 2550 6180 50  0000 C CNN
 F 2 "" H 2550 6000 50  0000 C CNN
@@
 $EndComp
 $Comp
-L +3V3 #PWR5
+L +3V3 #PWR018
 U 1 1 5887BB77
 P 2550 6300
-F 0 "#PWR5" H 2550 6150 50  0001 C CNN
+F 0 "#PWR018" H 2550 6150 50  0001 C CNN
 F 1 "+3V3" H 2550 6440 50  0000 C CNN
 F 2 "" H 2550 6300 50  0000 C CNN
@@
 	2550 6000 2550 6300
 $Comp
-L PWR_FLAG #FLG3
+L PWR_FLAG #FLG019
 U 1 1 5887BBDD
 P 3200 6000
-F 0 "#FLG3" H 3200 6095 50  0001 C CNN
+F 0 "#FLG019" H 3200 6095 50  0001 C CNN
 F 1 "PWR_FLAG" H 3200 6180 50  0000 C CNN
 F 2 "" H 3200 6000 50  0000 C CNN
@@
 $EndComp
 $Comp
-L GND #PWR8
+L GND #PWR020
 U 1 1 5887BC0C
 P 3200 6300
-F 0 "#PWR8" H 3200 6050 50  0001 C CNN
+F 0 "#PWR020" H 3200 6050 50  0001 C CNN
 F 1 "GND" H 3200 6150 50  0000 C CNN
 F 2 "" H 3200 6300 50  0000 C CNN
@@
 F 0 "P9" H 8950 4800 50  0000 C CNN
 F 1 "CONN_WS" V 9050 4550 50  0000 C CNN
-F 2 "Socket_Strips:Socket_Strip_Straight_1x04" H 8950 4550 50  0001 C CNN
+F 2 "Connectors_JST:JST_PH_B4B-PH-K_04x2.00mm_Straight" H 8950 4550 50  0001 C CNN
 F 3 "" H 8950 4550 50  0000 C CNN
 	1    8950 4550
@@
 WSTX
 $Comp
-L +5V #PWR19
+L +5V #PWR021
 U 1 1 5889449A
 P 8400 4600
-F 0 "#PWR19" H 8400 4450 50  0001 C CNN
+F 0 "#PWR021" H 8400 4450 50  0001 C CNN
 F 1 "+5V" H 8400 4740 50  0000 C CNN
 F 2 "" H 8400 4600 50  0000 C CNN
@@
 F 0 "P8" H 8800 2350 50  0000 C CNN
 F 1 "CONN_RB" V 8900 2100 50  0000 C CNN
-F 2 "Socket_Strips:Socket_Strip_Straight_1x04" H 8800 2100 50  0001 C CNN
+F 2 "Connectors_JST:JST_PH_B4B-PH-K_04x2.00mm_Straight" H 8800 2100 50  0001 C CNN
 F 3 "" H 8800 2100 50  0000 C CNN
 	1    8800 2100
@@
 RBTX
 $Comp
-L +5V #PWR18
+L +5V #PWR022
 U 1 1 588946C3
 P 8150 2150
-F 0 "#PWR18" H 8150 2000 50  0001 C CNN
+F 0 "#PWR022" H 8150 2000 50  0001 C CNN
 F 1 "+5V" H 8150 2290 50  0000 C CNN
 F 2 "" H 8150 2150 50  0000 C CNN
