File: weather-station/weather-station.sch (KiCad schematic (older format))
At the start: 17 parts, among them P1 CONN_01X05, P2 CONN_01X03, P3 CONN_01X02, P8 CONN_RB, U1 FUELGUAGE, U2 FEATHER, U3 pololu-vreg, U4 adafruit-solar-charger, U5 FEATHER

Commit message: Change RB connector footprint to 2.54mm pitch.
Parts:
- P8: footprint Connectors_JST:JST_PH_B4B-PH-K_04x2.00mm_Straight -> Socket_Strips:Socket_Strip_Straight_1x04_Pitch2.54mm
Changed lines of the file:
@@
 	1000 900  1200 900
 $Comp
-L PWR_FLAG #FLG04
+L PWR_FLAG #FLG03
 U 1 1 5887BA33
 P 9500 950
-F 0 "#FLG04" H 9500 1045 50  0001 C CNN
+F 0 "#FLG03" H 9500 1045 50  0001 C CNN
 F 1 "PWR_FLAG" H 9500 1130 50  0000 C CNN
 F 2 "" H 9500 950 50  0000 C CNN
@@
 $EndComp
 $Comp
-L +5V #PWR05
+L +5V #PWR04
 U 1 1 5887BA75
 P 9500 1250
-F 0 "#PWR05" H 9500 1100 50  0001 C CNN
+F 0 "#PWR04" H 9500 1100 50  0001 C CNN
 F 1 "+5V" H 9500 1390 50  0000 C CNN
 F 2 "" H 9500 1250 50  0000 C CNN
@@
 	9500 1250 9500 950
 $Comp
-L PWR_FLAG #FLG06
+L PWR_FLAG #FLG05
 U 1 1 5887BB48
 P 10100 950
-F 0 "#FLG06" H 10100 1045 50  0001 C CNN
+F 0 "#FLG05" H 10100 1045 50  0001 C CNN
 F 1 "PWR_FLAG" H 10100 1130 50  0000 C CNN
 F 2 "" H 10100 950 50  0000 C CNN
@@
 $EndComp
 $Comp
-L +3V3 #PWR07
+L +3V3 #PWR06
 U 1 1 5887BB77
 P 10100 1250
-F 0 "#PWR07" H 10100 1100 50  0001 C CNN
+F 0 "#PWR06" H 10100 1100 50  0001 C CNN
 F 1 "+3V3" H 10100 1390 50  0000 C CNN
 F 2 "" H 10100 1250 50  0000 C CNN
@@
 	10100 950  10100 1250
 $Comp
-L PWR_FLAG #FLG08
+L PWR_FLAG #FLG07
 U 1 1 5887BBDD
 P 10750 950
-F 0 "#FLG08" H 10750 1045 50  0001 C CNN
+F 0 "#FLG07" H 10750 1045 50  0001 C CNN
 F 1 "PWR_FLAG" H 10750 1130 50  0000 C CNN
 F 2 "" H 10750 950 50  0000 C CNN
@@
 $EndComp
 $Comp
-L GND #PWR09
+L GND #PWR08
 U 1 1 5887BC0C
 P 10750 1250
-F 0 "#PWR09" H 10750 1000 50  0001 C CNN
+F 0 "#PWR08" H 10750 1000 50  0001 C CNN
 F 1 "GND" H 10750 1100 50  0000 C CNN
 F 2 "" H 10750 1250 50  0000 C CNN
@@
 F 0 "P8" H 5350 1950 50  0000 C CNN
 F 1 "CONN_RB" V 5450 1700 50  0000 C CNN
-F 2 "Connectors_JST:JST_PH_B4B-PH-K_04x2.00mm_Straight" H 5350 1700 50  0001 C CNN
+F 2 "Socket_Strips:Socket_Strip_Straight_1x04_Pitch2.54mm" H 5350 1700 50  0001 C CNN
 F 3 "" H 5350 1700 50  0000 C CNN
 	1    5350 1700
@@
 RB_TX
 $Comp
-L +5V #PWR010
+L +5V #PWR09
 U 1 1 588946C3
 P 4700 1750
-F 0 "#PWR010" H 4700 1600 50  0001 C CNN
+F 0 "#PWR09" H 4700 1600 50  0001 C CNN
 F 1 "+5V" H 4700 1890 50  0000 C CNN
 F 2 "" H 4700 1750 50  0000 C CNN
@@
 $EndComp
 $Comp
-L GND #PWR011
+L GND #PWR010
 U 1 1 58C2D5B5
 P 1900 4600
-F 0 "#PWR011" H 1900 4350 50  0001 C CNN
+F 0 "#PWR010" H 1900 4350 50  0001 C CNN
 F 1 "GND" H 1900 4450 50  0000 C CNN
 F 2 "" H 1900 4600 50  0000 C CNN
@@
 B-
 $Comp
-L GND #PWR012
+L GND #PWR011
 U 1 1 58C2E2DD
 P 2700 2900
-F 0 "#PWR012" H 2700 2650 50  0001 C CNN
+F 0 "#PWR011" H 2700 2650 50  0001 C CNN
 F 1 "GND" H 2700 2750 50  0000 C CNN
 F 2 "" H 2700 2900 50  0000 C CNN
@@
 VLOAD
 $Comp
-L +5V #PWR013
+L +5V #PWR012
 U 1 1 58C2E77B
 P 3150 1900
-F 0 "#PWR013" H 3150 1750 50  0001 C CNN
+F 0 "#PWR012" H 3150 1750 50  0001 C CNN
 F 1 "+5V" H 3150 2040 50  0000 C CNN
 F 2 "" H 3150 1900 50  0000 C CNN
@@
 	3350 1700 3000 1700
 $Comp
-L GND #PWR014
+L GND #PWR013
 U 1 1 58C2E874
 P 2850 1800
-F 0 "#PWR014" H 2850 1550 50  0001 C CNN
+F 0 "#PWR013" H 2850 1550 50  0001 C CNN
 F 1 "GND" H 2850 1650 50  0000 C CNN
 F 2 "" H 2850 1800 50  0000 C CNN
@@
 	10400 4800 11100 4800
 $Comp
-L GND #PWR015
+L GND #PWR014
 U 1 1 58C2EED0
 P 8550 4600
-F 0 "#PWR015" H 8550 4350 50  0001 C CNN
+F 0 "#PWR014" H 8550 4350 50  0001 C CNN
 F 1 "GND" H 8550 4450 50  0000 C CNN
 F 2 "" H 8550 4600 50  0000 C CNN
@@
 NoConn ~ 7500 5550
 $Comp
-L GND #PWR016
+L GND #PWR015
 U 1 1 58C331D2
 P 8200 5100
-F 0 "#PWR016" H 8200 4850 50  0001 C CNN
+F 0 "#PWR015" H 8200 4850 50  0001 C CNN
 F 1 "GND" H 8200 4950 50  0000 C CNN
 F 2 "" H 8200 5100 50  0000 C CNN
@@
 3V3_WS
 $Comp
-L GND #PWR017
+L GND #PWR016
 U 1 1 58C3FF6A
 P 9950 3450
-F 0 "#PWR017" H 9950 3200 50  0001 C CNN
+F 0 "#PWR016" H 9950 3200 50  0001 C CNN
 F 1 "GND" H 9950 3300 50  0000 C CNN
 F 2 "" H 9950 3450 50  0000 C CNN
@@
 3V3_WS
 $Comp
-L PWR_FLAG #FLG018
+L PWR_FLAG #FLG017
 U 1 1 58C40491
 P 8750 950
-F 0 "#FLG018" H 8750 1045 50  0001 C CNN
+F 0 "#FLG017" H 8750 1045 50  0001 C CNN
 F 1 "PWR_FLAG" H 8750 1130 50  0000 C CNN
 F 2 "" H 8750 950 50  0000 C CNN
@@
 Connection ~ 10950 4800
 $Comp
-L GND #PWR019
+L GND #PWR018
 U 1 1 58C40D17
 P 10950 4150
-F 0 "#PWR019" H 10950 3900 50  0001 C CNN
+F 0 "#PWR018" H 10950 3900 50  0001 C CNN
 F 1 "GND" H 10950 4000 50  0000 C CNN
 F 2 "" H 10950 4150 50  0000 C CNN
@@
 3V3_WS
 $Comp
-L GND #PWR020
+L GND #PWR019
 U 1 1 58C42F4A
 P 9900 2700
-F 0 "#PWR020" H 9900 2450 50  0001 C CNN
+F 0 "#PWR019" H 9900 2450 50  0001 C CNN
 F 1 "GND" H 9900 2550 50  0000 C CNN
 F 2 "" H 9900 2700 50  0000 C CNN
@@
 	8600 4900 9050 4900
 $Comp
-L GND #PWR021
+L GND #PWR020
 U 1 1 58C4386D
 P 4700 6600
-F 0 "#PWR021" H 4700 6350 50  0001 C CNN
+F 0 "#PWR020" H 4700 6350 50  0001 C CNN
 F 1 "GND" H 4700 6450 50  0000 C CNN
 F 2 "" H 4700 6600 50  0000 C CNN
@@
 	4700 6600 4700 6500
 $Comp
-L GND #PWR022
+L GND #PWR021
 U 1 1 58C43E77
 P 4400 6600
-F 0 "#PWR022" H 4400 6350 50  0001 C CNN
+F 0 "#PWR021" H 4400 6350 50  0001 C CNN
 F 1 "GND" H 4400 6450 50  0000 C CNN
 F 2 "" H 4400 6600 50  0000 C CNN
@@
 	4400 6600 4400 6500
 $Comp
-L GND #PWR023
+L GND #PWR022
 U 1 1 58C43EB3
 P 4100 6600
-F 0 "#PWR023" H 4100 6350 50  0001 C CNN
+F 0 "#PWR022" H 4100 6350 50  0001 C CNN
 F 1 "GND" H 4100 6450 50  0000 C CNN
 F 2 "" H 4100 6600 50  0000 C CNN
@@
 	2600 2650 3350 2650
 $Comp
-L +3V3 #PWR?
+L +3V3 #PWR023
 U 1 1 58D46344
 P 800 1050
-F 0 "#PWR?" H 800 900 50  0001 C CNN
+F 0 "#PWR023" H 800 900 50  0001 C CNN
 F 1 "+3V3" H 800 1190 50  0000 C CNN
 F 2 "" H 800 1050 50  0000 C CNN
@@
 	800  1050 1200 1050
 $Comp
-L +3V3 #PWR?
+L +3V3 #PWR024
 U 1 1 58D46C53
 P 1800 4400
-F 0 "#PWR?" H 1800 4250 50  0001 C CNN
+F 0 "#PWR024" H 1800 4250 50  0001 C CNN
 F 1 "+3V3" H 1800 4540 50  0000 C CNN
 F 2 "" H 1800 4400 50  0000 C CNN
